File: EAGLE/KlingelESP32/KlingelESP32V1.brd (EAGLE design)
At the start: 46.7 x 80 mm, 29 parts, among them IC1 ESP-12E/F, J1 796683-2, J2 796683-2, J3 796683-2, J4 796683-2, Q1 AO3401

Commit message: Another error in VCC usage...
Connections:
- removed net VCC: R1.2
- net 3V3: now also R1.2
Changed lines of the file:
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@@
 <contactref element="C3" pad="1"/>
 <contactref element="R4" pad="2"/>
+<contactref element="R1" pad="2"/>
+<wire x1="27.94" y1="46.533" x2="27.94" y2="49.2" width="0" layer="19" extent="1-1"/>
+<wire x1="21.59" y1="44.77" x2="27.94" y2="46.533" width="0" layer="19" extent="1-1"/>
+<wire x1="11.43" y1="45.4" x2="21.59" y2="44.77" width="0" layer="19" extent="1-1"/>
 <wire x1="7.62" y1="44.45" x2="11.43" y2="45.4" width="0" layer="19" extent="1-1"/>
 <wire x1="4.13" y1="50.8" x2="7.62" y2="44.45" width="0" layer="19" extent="1-1"/>
 <wire x1="2.54" y1="54.61" x2="4.13" y2="50.8" width="0" layer="19" extent="1-1"/>
 <wire x1="7.29" y1="57.03" x2="2.54" y2="54.61" width="0" layer="19" extent="1-1"/>
-<wire x1="21.59" y1="44.77" x2="7.62" y2="44.45" width="0" layer="19" extent="1-1"/>
-<wire x1="27.94" y1="46.533" x2="21.59" y2="44.77" width="0" layer="19" extent="1-1"/>
-<wire x1="27.94" y1="49.2" x2="27.94" y2="46.533" width="0" layer="19" extent="1-1"/>
+<wire x1="16.19" y1="30.48" x2="21.59" y2="44.77" width="0" layer="19" extent="1-1"/>
 </signal>
 <signal name="RST">
@@
 <wire x1="20.32" y1="17.61" x2="28.89" y2="38.1" width="0" layer="19" extent="1-1"/>
 </signal>
-<signal name="VCC">
-<contactref element="R1" pad="2"/>
-</signal>
 <signal name="IO14">
